File: hardware/DC27-peripheral/DC27Audio.sch (KiCad schematic (older format))
At the start: 15 parts, among them J3 AudioJack3_Ground, J4 Conn_01x06_Female, U7 CS4344-CZZ

Commit message: commit the current hardware files
Parts:
- removed J4: Conn_01x06_Female, symbol Connector:Conn_01x06_Female
- C17, C18, C19, C20, C21, C22, C23: footprint (none) -> Capacitor_SMD:C_0603_1608Metric
- J3: footprint (none) -> Connector_Audio:Jack_Horizontal
- L3: footprint (none) -> Inductor_SMD:L_0603_1608Metric
- R12, R13, R14, R15: footprint (none) -> Resistor_SMD:R_0603_1608Metric
- U7: footprint SOP50P490X110-10N -> Housings_SSOP:TSSOP-10_3x3mm_Pitch0.5mm
Connections:
- net labels added: SND_LRCLK, SND_MCLK, SND_SCLK, SND_SDIN
- net labels removed: VCCIN
- wire segments 63 -> 52
Other:
- note removed: "GND"
- note removed: "LRCK\n\n"
- note removed: "MCLK\n"
- note removed: "SCLK"
- note removed: "SDIN\n"
- note removed: "VCC"
Changed lines of the file:
@@
 EESchema Schematic File Version 4
-LIBS:DC27-peripheral-cache
+LIBS:DC27-badge-cache
 EELAYER 26 0
 EELAYER END
@@
 	6500 3500 6850 3500
 Wire Wire Line
-	4350 3850 4350 4450
-$Comp
-L power:GND #PWR?
-U 1 1 5BA1588E
-P 4350 4450
-AR Path="/5BA1588E" Ref="#PWR?"  Part="1"
-AR Path="/5BA15261/5BA1588E" Ref="#PWR030"  Part="1"
-F 0 "#PWR030" H 4350 4200 50  0001 C CNN
-F 1 "GND" H 4355 4277 50  0000 C CNN
-F 2 "" H 4350 4450 50  0001 C CNN
-F 3 "" H 4350 4450 50  0001 C CNN
-	1    4350 4450
-	1    0    0    -1
-$EndComp
-Wire Wire Line
-	4250 3850 4350 3850
-Wire Wire Line
-	4650 3500 5100 3500
-Wire Wire Line
-	4650 3750 4650 3500
-Wire Wire Line
-	4250 3750 4650 3750
-Wire Wire Line
-	5000 3650 4250 3650
-Wire Wire Line
-	5000 3600 5000 3650
-Wire Wire Line
-	5100 3600 5000 3600
-Wire Wire Line
-	4900 3700 5100 3700
-Wire Wire Line
-	4900 3550 4900 3700
-Wire Wire Line
-	4250 3550 4900 3550
-Wire Wire Line
-	4750 3800 5100 3800
-Wire Wire Line
-	4750 3450 4750 3800
-Wire Wire Line
-	4250 3450 4750 3450
-Wire Wire Line
 	5000 4350 5000 4450
 Connection ~ 6600 4400
@@
 Wire Wire Line
 	6500 3900 6600 3900
-Wire Wire Line
-	4250 3950 4450 3950
-Text GLabel 4450 3950 2    50   Output ~ 0
-VCCIN
 Text GLabel 3000 2350 0    50   Input ~ 0
 VCC5V
@@
 F 0 "R13" V 7495 3950 50  0000 C CNN
 F 1 "470" V 7586 3950 50  0000 C CNN
-F 2 "" V 7740 3940 50  0001 C CNN
+F 2 "Resistor_SMD:R_0603_1608Metric" V 7740 3940 50  0001 C CNN
 F 3 "~" H 7700 3950 50  0001 C CNN
 	1    7700 3950
@@
 F 0 "R15" H 7432 4504 50  0000 R CNN
 F 1 "10K" H 7432 4595 50  0000 R CNN
-F 2 "" V 7540 4540 50  0001 C CNN
+F 2 "Resistor_SMD:R_0603_1608Metric" V 7540 4540 50  0001 C CNN
 F 3 "~" H 7500 4550 50  0001 C CNN
 	1    7500 4550
@@
 F 0 "R14" H 7450 4500 50  0000 L CNN
 F 1 "10K" H 7450 4600 50  0000 L CNN
-F 2 "" V 7390 4540 50  0001 C CNN
+F 2 "Resistor_SMD:R_0603_1608Metric" V 7390 4540 50  0001 C CNN
 F 3 "~" H 7350 4550 50  0001 C CNN
 	1    7350 4550
@@
 F 0 "R12" V 7495 3500 50  0000 C CNN
 F 1 "470" V 7586 3500 50  0000 C CNN
-F 2 "" V 7740 3490 50  0001 C CNN
+F 2 "Resistor_SMD:R_0603_1608Metric" V 7740 3490 50  0001 C CNN
 F 3 "~" H 7700 3500 50  0001 C CNN
 	1    7700 3500
@@
 F 0 "C21" V 6848 3950 50  0000 C CNN
 F 1 "3.3uF" V 6939 3950 50  0000 C CNN
-F 2 "" H 7138 3800 50  0001 C CNN
+F 2 "Capacitor_SMD:C_0603_1608Metric" H 7138 3800 50  0001 C CNN
 F 3 "~" H 7100 3950 50  0001 C CNN
 	1    7100 3950
@@
 F 0 "C20" V 6748 3500 50  0000 C CNN
 F 1 "3.3uF" V 6839 3500 50  0000 C CNN
-F 2 "" H 7038 3350 50  0001 C CNN
+F 2 "Capacitor_SMD:C_0603_1608Metric" H 7038 3350 50  0001 C CNN
 F 3 "~" H 7000 3500 50  0001 C CNN
 	1    7000 3500
@@
 F 0 "J3" H 8417 3529 50  0000 R CNN
 F 1 "AudioJack3_Ground" H 8417 3620 50  0000 R CNN
-F 2 "" H 8650 3600 50  0001 C CNN
+F 2 "Connector_Audio:Jack_Horizontal" H 8650 3600 50  0001 C CNN
 F 3 "~" H 8650 3600 50  0001 C CNN
 	1    8650 3600
@@
 F 0 "C23" H 6350 4250 50  0000 L CNN
 F 1 "10uF" H 6300 4150 50  0000 L CNN
-F 2 "" H 6638 4050 50  0001 C CNN
+F 2 "Capacitor_SMD:C_0603_1608Metric" H 6638 4050 50  0001 C CNN
 F 3 "~" H 6600 4200 50  0001 C CNN
 	1    6600 4200
@@
 F 0 "C22" H 5115 4246 50  0000 L CNN
 F 1 "3.3uF" H 5115 4155 50  0000 L CNN
-F 2 "" H 5038 4050 50  0001 C CNN
+F 2 "Capacitor_SMD:C_0603_1608Metric" H 5038 4050 50  0001 C CNN
 F 3 "~" H 5000 4200 50  0001 C CNN
 	1    5000 4200
@@
 F 0 "L3" V 4125 2350 50  0000 C CNN
 F 1 "L_Core_Ferrite" V 4034 2350 50  0000 C CNN
-F 2 "" H 3900 2350 50  0001 C CNN
+F 2 "Inductor_SMD:L_0603_1608Metric" H 3900 2350 50  0001 C CNN
 F 3 "~" H 3900 2350 50  0001 C CNN
 	1    3900 2350
@@
 F 0 "C17" H 3715 2696 50  0000 L CNN
 F 1 "0.1uF" H 3715 2605 50  0000 L CNN
-F 2 "" H 3638 2500 50  0001 C CNN
+F 2 "Capacitor_SMD:C_0603_1608Metric" H 3638 2500 50  0001 C CNN
 F 3 "~" H 3600 2650 50  0001 C CNN
 	1    3600 2650
@@
 F 0 "C19" H 4815 2696 50  0000 L CNN
 F 1 "0.1uF" H 4815 2605 50  0000 L CNN
-F 2 "" H 4738 2500 50  0001 C CNN
+F 2 "Capacitor_SMD:C_0603_1608Metric" H 4738 2500 50  0001 C CNN
 F 3 "~" H 4700 2650 50  0001 C CNN
 	1    4700 2650
@@
 F 0 "C18" H 4315 2696 50  0000 L CNN
 F 1 "0.1uF" H 4315 2605 50  0000 L CNN
-F 2 "" H 4238 2500 50  0001 C CNN
+F 2 "Capacitor_SMD:C_0603_1608Metric" H 4238 2500 50  0001 C CNN
 F 3 "~" H 4200 2650 50  0001 C CNN
 	1    4200 2650
 	1    0    0    -1
-$EndComp
-Text Notes 3800 4000 0    50   ~ 0
-VCC
-Text Notes 3800 3900 0    50   ~ 0
-GND
-Text Notes 3800 3800 0    50   ~ 0
-SDIN\n
-Text Notes 3800 3700 0    50   ~ 0
-SCLK
-Text Notes 3800 3700 0    50   ~ 0
-LRCK\n\n
-Text Notes 3800 3500 0    50   ~ 0
-MCLK\n
-$Comp
-L Connector:Conn_01x06_Female J?
-U 1 1 5BA1593D
-P 4050 3650
-AR Path="/5BA1593D" Ref="J?"  Part="1"
-AR Path="/5BA15261/5BA1593D" Ref="J4"  Part="1"
-F 0 "J4" H 3950 4100 50  0000 C CNN
-F 1 "Conn_01x06_Female" H 3950 4000 50  0000 C CNN
-F 2 "" H 4050 3650 50  0001 C CNN
-F 3 "~" H 4050 3650 50  0001 C CNN
-	1    4050 3650
-	-1   0    0    -1
 $EndComp
 $Comp
@@
 F 0 "U7" H 5800 3765 50  0000 C CNN
 F 1 "CS4344-CZZ" H 5800 3674 50  0000 C CNN
-F 2 "SOP50P490X110-10N" H 6350 3600 50  0001 L CNN
+F 2 "Housings_SSOP:TSSOP-10_3x3mm_Pitch0.5mm" H 6350 3600 50  0001 L CNN
 F 3 "http://uk.rs-online.com/web/p/products/4915754" H 6350 3500 50  0001 L CNN
 F 4 "Audio D/A Converter ICs Stereo DAC 24-Bit 192kHz" H 6350 3400 50  0001 L CNN "Description"
@@
 	1    0    0    -1
 $EndComp
+Text GLabel 4750 3800 0    50   Input ~ 0
+SND_MCLK
+Text GLabel 4750 3700 0    50   Input ~ 0
+SND_LRCLK
+Text GLabel 4750 3600 0    50   Input ~ 0
+SND_SCLK
+Text GLabel 4750 3500 0    50   Input ~ 0
+SND_SDIN
+Wire Wire Line
+	4750 3500 5100 3500
+Wire Wire Line
+	5100 3600 4750 3600
+Wire Wire Line
+	4750 3700 5100 3700
+Wire Wire Line
+	5100 3800 4750 3800
 $EndSCHEMATC

Commit message: Clean up SPI bus, set correct pins, start working through DRC errors.
Connections:
- net labels added: SND_LRCK, VCC_5V
- net labels removed: SND_LRCLK, VCC5V
Other:
- note added: "DC 27 Badge - Team Ides - John Adams / Bill Paul"
Changed lines of the file:
@@
 Wire Wire Line
 	6500 3900 6600 3900
-Text GLabel 3000 2350 0    50   Input ~ 0
-VCC5V
 $Comp
 L Device:R_US R?
@@
 	6600 3600 6500 3600
 Text GLabel 6600 3600 2    50   Input ~ 0
-VA
-Text GLabel 5200 2350 2    50   Output ~ 0
 VA
 Wire Wire Line
@@
 	1    0    0    -1
 $EndComp
-Text GLabel 4750 3800 0    50   Input ~ 0
+Wire Wire Line
+	4750 3500 5100 3500
+Wire Wire Line
+	5100 3600 4750 3600
+Wire Wire Line
+	4750 3700 5100 3700
+Wire Wire Line
+	5100 3800 4750 3800
+Text HLabel 4750 3500 0    50   Input ~ 0
+SND_SDIN
+Text HLabel 4750 3600 0    50   Input ~ 0
+SND_SCLK
+Text HLabel 4750 3700 0    50   Input ~ 0
+SND_LRCK
+Text HLabel 4750 3800 0    50   Input ~ 0
 SND_MCLK
-Text GLabel 4750 3700 0    50   Input ~ 0
-SND_LRCLK
-Text GLabel 4750 3600 0    50   Input ~ 0
-SND_SCLK
-Text GLabel 4750 3500 0    50   Input ~ 0
-SND_SDIN
-Wire Wire Line
-	4750 3500 5100 3500
-Wire Wire Line
-	5100 3600 4750 3600
-Wire Wire Line
-	4750 3700 5100 3700
-Wire Wire Line
-	5100 3800 4750 3800
+Text HLabel 3000 2350 0    50   Input ~ 0
+VCC_5V
+Text GLabel 5200 2350 2    50   Output ~ 0
+VA
+Text Notes 7350 7500 0    50   ~ 0
+DC 27 Badge - Team Ides - John Adams / Bill Paul
 $EndSCHEMATC

Commit message: update badge schematic with new pins, verify every pin
Parts:
- removed J3: AudioJack3_Ground, Connector_Audio:Jack_Horizontal, symbol Connector:AudioJack3_Ground
- added U10: TDA1308, symbol Amplifier_Audio:TDA1308
Connections:
- net labels added: AUDIO_OUT_L, AUDIO_OUT_R, VCC
- wire segments 52 -> 48
Other:
- note added: "40mW Audio Amplifer\n"
- note added: "Audio Power Filtering\n"
- note added: "I2S/I2C DAC"

Commit message: checkpoint all of the kicad stuff
Parts:
- removed C17, C19: 0.1uF, Capacitor_SMD:C_0603_1608Metric, symbol Device:C
- removed C20, C21, C22: 3.3uF, Capacitor_SMD:C_0603_1608Metric, symbol Device:C
- removed C23: 10uF, Capacitor_SMD:C_0603_1608Metric, symbol Device:C
- removed L3: L_Core_Ferrite, Inductor_SMD:L_0603_1608Metric, symbol Device:L_Core_Ferrite
- removed U10: TDA1308, symbol Amplifier_Audio:TDA1308
- added C23: 1mF, symbol Device:CP1
- added C24, C28: 0.1uF, Capacitor_SMD:C_0603_1608Metric, symbol Device:C
- added C25: 10mF Tantalum, Capacitor_SMD:C_0603_1608Metric, symbol Device:C
- added C26, C27, C29: 3.3uF, symbol Device:CP1
- added C30: 10uF, symbol Device:CP1
- added C31: 1uF Ceramic, symbol Device:C
- added J6: SPK LEFT, symbol Connector:Conn_01x02_Female
- added J7: SPK_RIGHT, symbol Connector:Conn_01x02_Female
- added R14, R19: 20K, symbol Device:R
- added U10: LM4929, symbol DC27-peripheral-cache:LM4929
- renumbered C18 to C22, R12 to R15, R13 to R16, R14 to R17, R15 to R18, U7 to U9
Connections:
- net labels removed: AUDIO_OUT_L, AUDIO_OUT_R, VA, VCC
- wire segments 48 -> 87
Other:
- note added: "+\n"
- note added: "CE20-14M-8 micro speaker x 2\n(0.25W to 0.5W max)\n"
- note added: "MUST PUT ALL OF THIS CIRCUITRY ON SEPARATE AREA OF BOARD WITH GROUND MOAT / 0 OHM\n RESISTOR, ETC."
- note added: "This circuit is turn-on pop guard\n"

Commit message: checkpoint everything - schematic passing DRC
Parts:
- removed C25: 10mF Tantalum, Capacitor_SMD:C_0603_1608Metric, symbol Device:C
- removed R17, R18: 10K, Resistor_SMD:R_0603_1608Metric, symbol Device:R_US
- removed U10: LM4929, symbol DC27-peripheral-cache:LM4929
- added C505, C510: 100uF, Capacitor_SMD:C_0603_1608Metric, symbol Device:CP1_Small
- added U502: LM4880, Package_SO:SOIC-8_3.9x4.9mm_P1.27mm, symbol LM4880:LM4880
- C502: renamed from C23; footprint (none) -> Capacitor_SMD:C_0603_1608Metric
- C504: renamed from C26; footprint (none) -> Capacitor_SMD:C_0603_1608Metric
- C506: renamed from C27; footprint (none) -> Capacitor_SMD:C_0603_1608Metric
- C508: renamed from C29; footprint (none) -> Capacitor_SMD:C_0603_1608Metric
- C509: renamed from C30; footprint (none) -> Capacitor_SMD:C_0603_1608Metric
- C511: renamed from C31; footprint (none) -> Capacitor_SMD:C_0603_1608Metric
- J501: renamed from J6; footprint (none) -> Connector_PinSocket_2.54mm:PinSocket_1x02_P2.54mm_Vertical_SMD_Pin1Left
- J502: renamed from J7; footprint (none) -> Connector_PinSocket_2.54mm:PinSocket_1x02_P2.54mm_Vertical_SMD_Pin1Left
- R501: renamed from R14; footprint (none) -> Resistor_SMD:R_0603_1608Metric
- R502: renamed from R15; value 470 -> 20K
- R503: renamed from R16; value 470 -> 20K
- R504: renamed from R19; footprint (none) -> Resistor_SMD:R_0603_1608Metric
- renumbered C22 to C501, C24 to C503, C28 to C507, U9 to U501
Connections:
- net labels added: +3.3V, AMP_SHUTDOWN
- net labels removed: VCC_5V
- wire segments 87 -> 72
Other:
- note added: "TBD- we don’t know what supply voltage to run this at\n"
- note removed: "40mW Audio Amplifer\n"
