File: hardware/DC27-peripheral/DC27LEDs.sch (KiCad schematic (older format))
At the start: 32 parts

Commit message: commit the current hardware files
Parts:
- D1, D10, D11, D12, D13, D14, D15, D16, D17, D18, D19, D2, D20, D21, D22, D23, D24, D25, D26, D27, D28, D29, D3, D30, D31, D32, D4, D5, D6, D7, D8, D9: footprint (none) -> LED_SMD:LED_Cree-PLCC4_3.2x2.8mm_CCW
Changed lines of the file:
@@
 EESchema Schematic File Version 4
-LIBS:DC27-peripheral-cache
+LIBS:DC27-badge-cache
 EELAYER 26 0
 EELAYER END
@@
 F 0 "D17" H 2500 4947 50  0000 C CNN
 F 1 "LED_ARGB" H 2500 4856 50  0000 C CNN
-F 2 "" H 2500 4400 50  0001 C CNN
+F 2 "LED_SMD:LED_Cree-PLCC4_3.2x2.8mm_CCW" H 2500 4400 50  0001 C CNN
 F 3 "~" H 2500 4400 50  0001 C CNN
 	1    2500 4450
@@
 F 0 "D18" H 3300 4947 50  0000 C CNN
 F 1 "LED_ARGB" H 3300 4856 50  0000 C CNN
-F 2 "" H 3300 4400 50  0001 C CNN
+F 2 "LED_SMD:LED_Cree-PLCC4_3.2x2.8mm_CCW" H 3300 4400 50  0001 C CNN
 F 3 "~" H 3300 4400 50  0001 C CNN
 	1    3300 4450
@@
 F 0 "D19" H 4200 4947 50  0000 C CNN
 F 1 "LED_ARGB" H 4200 4856 50  0000 C CNN
-F 2 "" H 4200 4400 50  0001 C CNN
+F 2 "LED_SMD:LED_Cree-PLCC4_3.2x2.8mm_CCW" H 4200 4400 50  0001 C CNN
 F 3 "~" H 4200 4400 50  0001 C CNN
 	1    4200 4450
@@
 F 0 "D20" H 5100 4947 50  0000 C CNN
 F 1 "LED_ARGB" H 5100 4856 50  0000 C CNN
-F 2 "" H 5100 4400 50  0001 C CNN
+F 2 "LED_SMD:LED_Cree-PLCC4_3.2x2.8mm_CCW" H 5100 4400 50  0001 C CNN
 F 3 "~" H 5100 4400 50  0001 C CNN
 	1    5100 4450
@@
 F 0 "D21" H 6100 4947 50  0000 C CNN
 F 1 "LED_ARGB" H 6100 4856 50  0000 C CNN
-F 2 "" H 6100 4400 50  0001 C CNN
+F 2 "LED_SMD:LED_Cree-PLCC4_3.2x2.8mm_CCW" H 6100 4400 50  0001 C CNN
 F 3 "~" H 6100 4400 50  0001 C CNN
 	1    6100 4450
@@
 F 0 "D22" H 7100 4947 50  0000 C CNN
 F 1 "LED_ARGB" H 7100 4856 50  0000 C CNN
-F 2 "" H 7100 4400 50  0001 C CNN
+F 2 "LED_SMD:LED_Cree-PLCC4_3.2x2.8mm_CCW" H 7100 4400 50  0001 C CNN
 F 3 "~" H 7100 4400 50  0001 C CNN
 	1    7100 4450
@@
 F 0 "D23" H 8050 4947 50  0000 C CNN
 F 1 "LED_ARGB" H 8050 4856 50  0000 C CNN
-F 2 "" H 8050 4400 50  0001 C CNN
+F 2 "LED_SMD:LED_Cree-PLCC4_3.2x2.8mm_CCW" H 8050 4400 50  0001 C CNN
 F 3 "~" H 8050 4400 50  0001 C CNN
 	1    8050 4450
@@
 F 0 "D24" H 9050 4947 50  0000 C CNN
 F 1 "LED_ARGB" H 9050 4856 50  0000 C CNN
-F 2 "" H 9050 4400 50  0001 C CNN
+F 2 "LED_SMD:LED_Cree-PLCC4_3.2x2.8mm_CCW" H 9050 4400 50  0001 C CNN
 F 3 "~" H 9050 4400 50  0001 C CNN
 	1    9050 4450
@@
 F 0 "D25" H 2500 6247 50  0000 C CNN
 F 1 "LED_ARGB" H 2500 6156 50  0000 C CNN
-F 2 "" H 2500 5700 50  0001 C CNN
+F 2 "LED_SMD:LED_Cree-PLCC4_3.2x2.8mm_CCW" H 2500 5700 50  0001 C CNN
 F 3 "~" H 2500 5700 50  0001 C CNN
 	1    2500 5750
@@
 F 0 "D26" H 3300 6247 50  0000 C CNN
 F 1 "LED_ARGB" H 3300 6156 50  0000 C CNN
-F 2 "" H 3300 5700 50  0001 C CNN
+F 2 "LED_SMD:LED_Cree-PLCC4_3.2x2.8mm_CCW" H 3300 5700 50  0001 C CNN
 F 3 "~" H 3300 5700 50  0001 C CNN
 	1    3300 5750
@@
 F 0 "D27" H 4200 6247 50  0000 C CNN
 F 1 "LED_ARGB" H 4200 6156 50  0000 C CNN
-F 2 "" H 4200 5700 50  0001 C CNN
+F 2 "LED_SMD:LED_Cree-PLCC4_3.2x2.8mm_CCW" H 4200 5700 50  0001 C CNN
 F 3 "~" H 4200 5700 50  0001 C CNN
 	1    4200 5750
@@
 F 0 "D28" H 5100 6247 50  0000 C CNN
 F 1 "LED_ARGB" H 5100 6156 50  0000 C CNN
-F 2 "" H 5100 5700 50  0001 C CNN
+F 2 "LED_SMD:LED_Cree-PLCC4_3.2x2.8mm_CCW" H 5100 5700 50  0001 C CNN
 F 3 "~" H 5100 5700 50  0001 C CNN
 	1    5100 5750
@@
 F 0 "D29" H 6100 6247 50  0000 C CNN
 F 1 "LED_ARGB" H 6100 6156 50  0000 C CNN
-F 2 "" H 6100 5700 50  0001 C CNN
+F 2 "LED_SMD:LED_Cree-PLCC4_3.2x2.8mm_CCW" H 6100 5700 50  0001 C CNN
 F 3 "~" H 6100 5700 50  0001 C CNN
 	1    6100 5750
@@
 F 0 "D30" H 7100 6247 50  0000 C CNN
 F 1 "LED_ARGB" H 7100 6156 50  0000 C CNN
-F 2 "" H 7100 5700 50  0001 C CNN
+F 2 "LED_SMD:LED_Cree-PLCC4_3.2x2.8mm_CCW" H 7100 5700 50  0001 C CNN
 F 3 "~" H 7100 5700 50  0001 C CNN
 	1    7100 5750
@@
 F 0 "D31" H 8050 6247 50  0000 C CNN
 F 1 "LED_ARGB" H 8050 6156 50  0000 C CNN
-F 2 "" H 8050 5700 50  0001 C CNN
+F 2 "LED_SMD:LED_Cree-PLCC4_3.2x2.8mm_CCW" H 8050 5700 50  0001 C CNN
 F 3 "~" H 8050 5700 50  0001 C CNN
 	1    8050 5750
@@
 F 0 "D32" H 9050 6247 50  0000 C CNN
 F 1 "LED_ARGB" H 9050 6156 50  0000 C CNN
-F 2 "" H 9050 5700 50  0001 C CNN
+F 2 "LED_SMD:LED_Cree-PLCC4_3.2x2.8mm_CCW" H 9050 5700 50  0001 C CNN
 F 3 "~" H 9050 5700 50  0001 C CNN
 	1    9050 5750
@@
 F 0 "D1" H 2450 1947 50  0000 C CNN
 F 1 "LED_ARGB" H 2450 1856 50  0000 C CNN
-F 2 "" H 2450 1400 50  0001 C CNN
+F 2 "LED_SMD:LED_Cree-PLCC4_3.2x2.8mm_CCW" H 2450 1400 50  0001 C CNN
 F 3 "~" H 2450 1400 50  0001 C CNN
 	1    2450 1450
@@
 F 0 "D2" H 3250 1947 50  0000 C CNN
 F 1 "LED_ARGB" H 3250 1856 50  0000 C CNN
-F 2 "" H 3250 1400 50  0001 C CNN
+F 2 "LED_SMD:LED_Cree-PLCC4_3.2x2.8mm_CCW" H 3250 1400 50  0001 C CNN
 F 3 "~" H 3250 1400 50  0001 C CNN
 	1    3250 1450
@@
 F 0 "D3" H 4150 1947 50  0000 C CNN
 F 1 "LED_ARGB" H 4150 1856 50  0000 C CNN
-F 2 "" H 4150 1400 50  0001 C CNN
+F 2 "LED_SMD:LED_Cree-PLCC4_3.2x2.8mm_CCW" H 4150 1400 50  0001 C CNN
 F 3 "~" H 4150 1400 50  0001 C CNN
 	1    4150 1450
@@
 F 0 "D4" H 5050 1947 50  0000 C CNN
 F 1 "LED_ARGB" H 5050 1856 50  0000 C CNN
-F 2 "" H 5050 1400 50  0001 C CNN
+F 2 "LED_SMD:LED_Cree-PLCC4_3.2x2.8mm_CCW" H 5050 1400 50  0001 C CNN
 F 3 "~" H 5050 1400 50  0001 C CNN
 	1    5050 1450
@@
 F 0 "D5" H 6050 1947 50  0000 C CNN
 F 1 "LED_ARGB" H 6050 1856 50  0000 C CNN
-F 2 "" H 6050 1400 50  0001 C CNN
+F 2 "LED_SMD:LED_Cree-PLCC4_3.2x2.8mm_CCW" H 6050 1400 50  0001 C CNN
 F 3 "~" H 6050 1400 50  0001 C CNN
 	1    6050 1450
@@
 F 0 "D6" H 7050 1947 50  0000 C CNN
 F 1 "LED_ARGB" H 7050 1856 50  0000 C CNN
-F 2 "" H 7050 1400 50  0001 C CNN
+F 2 "LED_SMD:LED_Cree-PLCC4_3.2x2.8mm_CCW" H 7050 1400 50  0001 C CNN
 F 3 "~" H 7050 1400 50  0001 C CNN
 	1    7050 1450
@@
 F 0 "D7" H 8000 1947 50  0000 C CNN
 F 1 "LED_ARGB" H 8000 1856 50  0000 C CNN
-F 2 "" H 8000 1400 50  0001 C CNN
+F 2 "LED_SMD:LED_Cree-PLCC4_3.2x2.8mm_CCW" H 8000 1400 50  0001 C CNN
 F 3 "~" H 8000 1400 50  0001 C CNN
 	1    8000 1450
@@
 F 0 "D8" H 9000 1947 50  0000 C CNN
 F 1 "LED_ARGB" H 9000 1856 50  0000 C CNN
-F 2 "" H 9000 1400 50  0001 C CNN
+F 2 "LED_SMD:LED_Cree-PLCC4_3.2x2.8mm_CCW" H 9000 1400 50  0001 C CNN
 F 3 "~" H 9000 1400 50  0001 C CNN
 	1    9000 1450
@@
 F 0 "D9" H 2450 3247 50  0000 C CNN
 F 1 "LED_ARGB" H 2450 3156 50  0000 C CNN
-F 2 "" H 2450 2700 50  0001 C CNN
+F 2 "LED_SMD:LED_Cree-PLCC4_3.2x2.8mm_CCW" H 2450 2700 50  0001 C CNN
 F 3 "~" H 2450 2700 50  0001 C CNN
 	1    2450 2750
@@
 F 0 "D10" H 3250 3247 50  0000 C CNN
 F 1 "LED_ARGB" H 3250 3156 50  0000 C CNN
-F 2 "" H 3250 2700 50  0001 C CNN
+F 2 "LED_SMD:LED_Cree-PLCC4_3.2x2.8mm_CCW" H 3250 2700 50  0001 C CNN
 F 3 "~" H 3250 2700 50  0001 C CNN
 	1    3250 2750
@@
 F 0 "D11" H 4150 3247 50  0000 C CNN
 F 1 "LED_ARGB" H 4150 3156 50  0000 C CNN
-F 2 "" H 4150 2700 50  0001 C CNN
+F 2 "LED_SMD:LED_Cree-PLCC4_3.2x2.8mm_CCW" H 4150 2700 50  0001 C CNN
 F 3 "~" H 4150 2700 50  0001 C CNN
 	1    4150 2750
@@
 F 0 "D12" H 5050 3247 50  0000 C CNN
 F 1 "LED_ARGB" H 5050 3156 50  0000 C CNN
-F 2 "" H 5050 2700 50  0001 C CNN
+F 2 "LED_SMD:LED_Cree-PLCC4_3.2x2.8mm_CCW" H 5050 2700 50  0001 C CNN
 F 3 "~" H 5050 2700 50  0001 C CNN
 	1    5050 2750
@@
 F 0 "D13" H 6050 3247 50  0000 C CNN
 F 1 "LED_ARGB" H 6050 3156 50  0000 C CNN
-F 2 "" H 6050 2700 50  0001 C CNN
+F 2 "LED_SMD:LED_Cree-PLCC4_3.2x2.8mm_CCW" H 6050 2700 50  0001 C CNN
 F 3 "~" H 6050 2700 50  0001 C CNN
 	1    6050 2750
@@
 F 0 "D14" H 7050 3247 50  0000 C CNN
 F 1 "LED_ARGB" H 7050 3156 50  0000 C CNN
-F 2 "" H 7050 2700 50  0001 C CNN
+F 2 "LED_SMD:LED_Cree-PLCC4_3.2x2.8mm_CCW" H 7050 2700 50  0001 C CNN
 F 3 "~" H 7050 2700 50  0001 C CNN
 	1    7050 2750
@@
 F 0 "D15" H 8000 3247 50  0000 C CNN
 F 1 "LED_ARGB" H 8000 3156 50  0000 C CNN
-F 2 "" H 8000 2700 50  0001 C CNN
+F 2 "LED_SMD:LED_Cree-PLCC4_3.2x2.8mm_CCW" H 8000 2700 50  0001 C CNN
 F 3 "~" H 8000 2700 50  0001 C CNN
 	1    8000 2750
@@
 F 0 "D16" H 9000 3247 50  0000 C CNN
 F 1 "LED_ARGB" H 9000 3156 50  0000 C CNN
-F 2 "" H 9000 2700 50  0001 C CNN
+F 2 "LED_SMD:LED_Cree-PLCC4_3.2x2.8mm_CCW" H 9000 2700 50  0001 C CNN
 F 3 "~" H 9000 2700 50  0001 C CNN
 	1    9000 2750

Commit message: Clean up SPI bus, set correct pins, start working through DRC errors.
Other:
- note added: "DC 27 Badge - Team Ides - John Adams / Bill Paul"
Changed lines of the file:
@@
 Text Notes 9600 800  0    50   ~ 10
 LEDs:\n1616 0603 RGB common anode\n
+Text Notes 7400 7500 0    50   ~ 0
+DC 27 Badge - Team Ides - John Adams / Bill Paul
 $EndSCHEMATC

Commit message: checkpoint everything - schematic passing DRC
Parts:
- renumbered D1 to D201, D2 to D202, D3 to D203, D4 to D204, D5 to D205, D6 to D206, D7 to D207, D8 to D208, D9 to D209, D10 to D210, D11 to D211, D12 to D212, D13 to D213, D14 to D214, D15 to D215, D16 to D216, D17 to D217, D18 to D218, D19 to D219, D20 to D220, D21 to D221, D22 to D222, D23 to D223, D24 to D224, D25 to D225, D26 to D226, D27 to D227, D28 to D228, D29 to D229, D30 to D230, D31 to D231, D32 to D232
Connections:
- wire segments 352 -> 350
Other:
- note added: "LEDs:\nMacrofab house part CREE PLCC4 / CLV1L-FKB - 23 cents @ 1"
- note removed: "LEDs:\n1616 0603 RGB common anode\n"
