File: hardware/DC27-peripheral/file5C2B533B.sch (KiCad schematic (older format))
At the start: 6 parts, among them U2 CP2102N-A01-GQFN28

Commit message: checkpoint everything - schematic passing DRC
Parts:
- removed C1: 10uF, symbol Device:C_Small
- removed C2: 0.1uF, symbol Device:C_Small
- added C601, C603: 10uF, Capacitor_SMD:C_1206_3216Metric, symbol Device:C
- added C602, C604: 0.1uF, Capacitor_SMD:C_0603_1608Metric, symbol Device:C
- added D601: TX LED, Diode_SMD:D_0603_1608Metric, symbol Device:LED
- added D602: RX LED, Diode_SMD:D_0603_1608Metric, symbol Device:LED
- added J601: USB_MICRO_RIGHT, MF_Connectors:MF_Connectors-MICROUSB-RIGHT, symbol MF_Connectors:USB_MICRO_RIGHT
- added L601, L602, L603: LXES15AAA1-153, Diode_SMD:D_01005_0402Metric, symbol jna_parts:LXES15AAA1-153
- added R602, R603: 47, Resistor_SMD:R_0603_1608Metric, symbol Device:R
- R601: renamed from R20; footprint (none) -> Resistor_SMD:R_0603_1608Metric
- R604: renamed from R21; value 47.5K -> 22.1k; footprint (none) -> Resistor_SMD:R_0603_1608Metric
- R605: renamed from R22; value 22.1k -> 47.5k; footprint (none) -> Resistor_SMD:R_0603_1608Metric
- U601: renamed from U2; footprint Package_DFN_QFN:QFN-24-1EP_4x4mm_P0.5mm_EP2.6x2.6mm -> Package_DFN_QFN:QFN-28-1EP_5x5mm_P0.5mm_EP3.35x3.35mm_ThermalVias
Connections:
- net labels added: VBUS
- net labels removed: UART_DTR
- wire segments 29 -> 77
- no-connect marks 4 -> 15
Other:
- note added: "DTR and DSR are not used in this design"
- note added: "ESD Protection\n"
- note added: "floating shield to reduce noise"
- note removed: "VREGIN is USB voltage, typically.\nVDD is an output line if the interal regulator is in use.\nHow much current can this chip source?\n"
