File: hardware/DC27-peripheral/DC27-badge.sch (KiCad schematic (older format))
At the start: 12 parts, among them J5 Conn_02x20_Odd_Even, J6 Conn_02x02_Counter_Clockwise, J7 Conn_ARM_JTAG_SWD_10, SW1 UP, SW2 DN, SW3 LEFT, SW4 RIGHT, SW5 A, SW6 B, SW7 RESET, U1 BMD-340-A-R

Commit message: commit the current hardware files
Parts:
- added R17, R18: 27k, Resistor_SMD:R_0603_1608Metric, symbol Device:R
- J5: footprint (none) -> Connector_PinHeader_1.00mm:PinHeader_2x20_P1.00mm_Vertical_SMD
- J6: footprint (none) -> Connector_PinHeader_1.00mm:PinHeader_2x02_P1.00mm_Vertical_SMD
- R16: footprint (none) -> Resistor_SMD:R_0603_1608Metric
- SW1, SW2, SW3, SW4, SW5, SW6, SW7: footprint MF_Switches_TACT4.2MM -> MF_Switches:MF_Switches-TACT4.2MM
- U1: footprint RIGADO_BMD-340-A-R -> BMD-340-A-R:RIGADO_BMD-340-A-R
Connections:
- wire segments 134 -> 140
- no-connect marks 29 -> 30
Other:
- note added: "13,14 are external XTAL\n"
- note added: "ESD protection on power schematic"
- note added: "PSELRESET[0] and PSELRESET[1] must be\n0x7fffffd2 for ~RESET"
- note added: "Shitty Add On - 1\n"
- note removed: "Shitty Add On!\n"

Commit message: Update the main schematic with pins from bill's changes
Parts:
- added C25, C26: 12pF, symbol Device:C
- added TP5: XTAL0, symbol Connector:TestPoint
- added TP6: XTAL1, symbol Connector:TestPoint
- added Y1: 32.768Khz XTAL, symbol Device:Crystal
Connections:
- net labels added: I2S_LRCK, I2S_MCK, I2S_SCLK, I2S_SDOUT, LED_2, LED_3, LED_4, NFC_ANT0, NFC_ANT1, QSPI_CLK, QSPI_CS, QSPI_DIO0, QSPI_DIO1, QSPI_DIO2, QSPI_DIO3, SCREEN_CD, SPI_MISO, SPI_MOSI, SPI_SCLK, UART_CTS, UART_RTS, UART_RX, UART_TX, XTAL0, XTAL1
- wire segments 140 -> 178
- no-connect marks 30 -> 42
Other:
- note added: "CLOCK\n"
- note added: "SPI\n"
- note removed: "13,14 are external XTAL\n"

Commit message: Clean up SPI bus, set correct pins, start working through DRC errors.
Parts:
- added TP7: SPI_MOSI, symbol Connector:TestPoint
- added TP8: SPI_MISO, symbol Connector:TestPoint
- added TP9: SPI_SCK, symbol Connector:TestPoint
Connections:
- net labels removed: SCREEN_CD
- wire segments 178 -> 197
Other:
- note added: "Things to get from Bill:\nQSPI usage / pinout / where does it go\nWhere is I2C? Is it enabled?\nWhere do I2S Pins go?\nDo we need NFC pins?\nWhich SPI Bus is display on?"
- note added: "populate with\nsmd flat-mount connector"
- note removed: "populate with\nsmd mount connector"
Changed lines of the file:
@@
 DC27 Audio Circuit\n
 $Sheet
-S 550  1500 1450 650
+S 550  1500 1200 650
 U 5BA1B02E
 F0 "LEDs" 50
@@
 $EndSheet
 $Sheet
-S 550  2350 1450 650
+S 550  2350 1200 650
 U 5BD866AF
 F0 "LED Interface" 50
@@
 $EndSheet
 $Sheet
-S 2100 650  1200 650
+S 550  650  1200 650
 U 5BA3F217
 F0 "DC Power" 50
@@
 $EndSheet
 $Sheet
-S 550  650  1450 650
+S 2700 650  900  650
 U 5BA15261
 F0 "DC27Audio" 50
 F1 "DC27Audio.sch" 50
+F2 "SND_SDIN" I L 2700 750 50
+F3 "SND_SCLK" I L 2700 900 50
+F4 "SND_LRCK" I L 2700 1050 50
+F5 "SND_MCLK" I L 2700 1200 50
+F6 "VCC_5V" I R 3600 750 50
 $EndSheet
 $Comp
@@
 NoConn ~ 10350 3000
 NoConn ~ 10350 2900
-Text Notes 8850 2300 0    50   ~ 10
+Text Notes 8900 2300 0    50   ~ 10
 DISPLAY\n
 Wire Notes Line
@@
 Wire Wire Line
 	10750 1400 10750 1250
-Text Notes 3550 700  0    50   ~ 10
+Text Notes 4100 600  0    50   ~ 10
 TODO: FTDI
-Text Notes 9150 4900 0    50   Italic 0
-populate with\nsmd mount connector
+Text Notes 8900 5100 0    50   Italic 0
+populate with\nsmd flat-mount connector
 $Comp
 L Device:R R17
@@
 NoConn ~ 4300 3550
 Text GLabel 4100 3750 0    50   Output ~ 0
-SCREEN_CD
+DISP_DC
 Wire Wire Line
 	4100 3650 4300 3650
@@
 NoConn ~ 5750 3350
 NoConn ~ 5750 3250
-Text GLabel 6000 2850 2    50   Output ~ 0
+Text GLabel 6150 2850 2    50   Output ~ 0
 I2S_SDOUT
-Wire Wire Line
-	5750 2850 6000 2850
-Text GLabel 6000 2950 2    50   Output ~ 0
+Text GLabel 6150 2950 2    50   Output ~ 0
 I2S_SCLK
-Wire Wire Line
-	5750 2950 6000 2950
-Text GLabel 6000 3050 2    50   Output ~ 0
+Text GLabel 6150 3050 2    50   Output ~ 0
 I2S_LRCK
-Wire Wire Line
-	5750 3050 6000 3050
-Text GLabel 6000 3150 2    50   Output ~ 0
+Text GLabel 6150 3150 2    50   Output ~ 0
 I2S_MCK
-Wire Wire Line
-	5750 3150 6000 3150
 $Comp
 L Connector:TestPoint TP6
@@
 Wire Notes Line
 	7400 500  7400 6550
-Text GLabel 7850 2700 0    50   Output ~ 0
+Text GLabel 7850 3550 0    50   Output ~ 0
 SPI_MISO
 Text GLabel 7850 4300 0    50   Input ~ 0
 SPI_SCLK
-Text GLabel 7850 3550 0    50   Input ~ 0
+Text GLabel 7850 2900 0    50   Input ~ 0
 SPI_MOSI
 Wire Notes Line
-	8800 2200 8800 5200
+	8850 2200 8850 5200
 Text Notes 7450 2300 0    50   ~ 10
 SPI\n
+Text GLabel 8150 2900 2    50   Input ~ 0
+DISP_SDI_MOSI
+Text GLabel 8150 3050 2    50   Input ~ 0
+SD_MOSI
+Wire Wire Line
+	7850 2900 8000 2900
+Wire Wire Line
+	8150 3050 8000 3050
+Wire Wire Line
+	8000 3050 8000 2900
+Connection ~ 8000 2900
+Text GLabel 8150 3550 2    50   Input ~ 0
+DISP_SDO_MOSI
+Wire Wire Line
+	7850 3550 8000 3550
+Text GLabel 8150 3700 2    50   Input ~ 0
+SD_MISO
+Wire Wire Line
+	8150 3700 8000 3700
+Wire Wire Line
+	8000 3700 8000 3550
+Connection ~ 8000 3550
+Wire Wire Line
+	8000 3550 8150 3550
+$Comp
+L Connector:TestPoint TP7
+U 1 1 5BE594F0
+P 8000 2700
+F 0 "TP7" H 8058 2820 50  0000 L CNN
+F 1 "SPI_MOSI" H 8058 2729 50  0000 L CNN
+F 2 "" H 8200 2700 50  0001 C CNN
+F 3 "~" H 8200 2700 50  0001 C CNN
+	1    8000 2700
+	1    0    0    -1
+$EndComp
+Wire Wire Line
+	8000 2900 8000 2700
+Wire Wire Line
+	8000 2900 8150 2900
+$Comp
+L Connector:TestPoint TP8
+U 1 1 5BE6D4D8
+P 8000 3350
+F 0 "TP8" H 8058 3470 50  0000 L CNN
+F 1 "SPI_MISO" H 8058 3379 50  0000 L CNN
+F 2 "" H 8200 3350 50  0001 C CNN
+F 3 "~" H 8200 3350 50  0001 C CNN
+	1    8000 3350
+	1    0    0    -1
+$EndComp
+Wire Wire Line
+	8000 3350 8000 3550
+Text GLabel 8150 4300 2    50   Output ~ 0
+SD_SCLK
+Text GLabel 8150 4500 2    50   Output ~ 0
+DISP_SCLK
+Wire Wire Line
+	7850 4300 8000 4300
+Wire Wire Line
+	8150 4500 8000 4500
+Wire Wire Line
+	8000 4500 8000 4300
+Connection ~ 8000 4300
+Wire Wire Line
+	8000 4300 8150 4300
+$Comp
+L Connector:TestPoint TP9
+U 1 1 5BE8BAC1
+P 8000 4150
+F 0 "TP9" H 8058 4270 50  0000 L CNN
+F 1 "SPI_SCK" H 8058 4179 50  0000 L CNN
+F 2 "" H 8200 4150 50  0001 C CNN
+F 3 "~" H 8200 4150 50  0001 C CNN
+	1    8000 4150
+	1    0    0    -1
+$EndComp
+Wire Wire Line
+	8000 4150 8000 4300
+Text Notes 4100 1150 0    50   ~ 0
+Things to get from Bill:\nQSPI usage / pinout / where does it go\nWhere is I2C? Is it enabled?\nWhere do I2S Pins go?\nDo we need NFC pins?\nWhich SPI Bus is display on?
+Wire Wire Line
+	5750 3150 6150 3150
+Wire Wire Line
+	5750 3050 6150 3050
+Wire Wire Line
+	5750 2950 6150 2950
+Wire Wire Line
+	5750 2850 6150 2850
+Text GLabel 2500 750  0    50   Input ~ 0
+I2S_SDOUT
+Text GLabel 2450 900  0    50   Input ~ 0
+I2S_SCLK
+Text GLabel 2450 1050 0    50   Input ~ 0
+I2S_LRCK
+Text GLabel 2450 1200 0    50   Input ~ 0
+I2S_MCK
+Wire Wire Line
+	2450 1200 2700 1200
+Wire Wire Line
+	2450 1050 2700 1050
+Wire Wire Line
+	2700 900  2450 900
+Wire Wire Line
+	2500 750  2700 750
 $EndSCHEMATC

Commit message: update badge schematic with new pins, verify every pin
Parts:
- removed R18: 27k, Resistor_SMD:R_0603_1608Metric, symbol Device:R
- added C27: 4.7uF, symbol Device:C
- added C28: 0.1uF, symbol Device:C
- added TP10: SDT_SPI_SCK, symbol Connector:TestPoint
- added TP11, TP12: DISP_MOSI, symbol Connector:TestPoint
- added U9: CP2102N-A01-GQFN24, Package_DFN_QFN:QFN-24-1EP_4x4mm_P0.5mm_EP2.6x2.6mm, symbol Interface_USB:CP2102N-A01-GQFN24
- R17: value 27k -> R; footprint Resistor_SMD:R_0603_1608Metric -> (none)
- TP7: value SPI_MOSI -> SDT_SPI_MOSI
- TP8: value SPI_MISO -> SDT_SPI_MISO
- TP9: value SPI_SCK -> SDT_SPI_SCK
Connections:
- net labels added: DISP_MISO, DISP_MOSI, I2C_SCK, I2C_SDA, SCREEN_SPI_MISO, SCREEN_SPI_MOSI, SCREEN_SPI_SCLK, SDT_SPI_MISO, SDT_SPI_MOSI, SDT_SPI_SCK
- net labels removed: DISP_SDI_MOSI, DISP_SDO_MOSI, I2C1_SCL, I2C1_SDA, SPI_MISO, SPI_MOSI, SPI_SCLK
- wire segments 197 -> 221
- no-connect marks 42 -> 43
Other:
- note added: "FTDI/USB CONSOLE"
- note added: "SPI BUS 3\n"
- note added: "Things to get from Bill:\nQSPI usage / pinout / where does it go\nWhere is I2C? Is it enabled?\nWhere do I2S Pins go?\nDo we need NFC pins?\nWhich SPI Bus is display on?\n\nIssue with cp2012n is it's sensitivity on vbus detect pin. If > 5.8v = boom"
- note removed: "TODO: FTDI"
- note removed: "Things to get from Bill:\nQSPI usage / pinout / where does it go\nWhere is I2C? Is it enabled?\nWhere do I2S Pins go?\nDo we need NFC pins?\nWhich SPI Bus is display on?"

Commit message: checkpoint all of the kicad stuff
Parts:
- removed C27: 4.7uF, symbol Device:C
- removed C28: 0.1uF, symbol Device:C
- removed R17: R, symbol Device:R
- removed U9: CP2102N-A01-GQFN24, Package_DFN_QFN:QFN-24-1EP_4x4mm_P0.5mm_EP2.6x2.6mm, symbol Interface_USB:CP2102N-A01-GQFN24
- added J8: Conn_01x02_Female, symbol Connector:Conn_01x02_Female
- added SW8: RESET, MF_Switches:MF_Switches-TACT4.2MM, symbol MF_Switches:TACT_4.2MM
- renumbered C25 to C3, C26 to C4, J6 to J1, J5 to J2, J7 to J3, R16 to R1, TP7 to TP1, TP8 to TP2, TP9 to TP3, TP10 to TP4, TP11 to TP5, TP12 to TP6, TP5 to TP7, TP6 to TP8
Connections:
- net labels added: ~ENTER
- net labels removed: LED_2, LED_3, LED_4, QSPI_CLK, QSPI_CS, QSPI_DIO0, QSPI_DIO1, QSPI_DIO2, QSPI_DIO3, USBDATA+, USBDATA-
- wire segments 221 -> 212
- no-connect marks 43 -> 47
Other:
- note added: "Am very unsure about this layout."
- note added: "NFC antenna connector - DNP"
- note added: "p0.14 = led 2\np0.15 = led 3\np0.16 = led 4 on dev board\n"
- note removed: "FTDI/USB CONSOLE"

Commit message: checkpoint everything - schematic passing DRC
Parts:
- removed J1: Conn_02x02_Counter_Clockwise, Connector_PinHeader_1.00mm:PinHeader_2x02_P1.00mm_Vertical_SMD, symbol Connector_Generic:Conn_02x02_Counter_Clockwise
- added J102: ShittyAddOnL, Connector_PinSocket_2.54mm:PinSocket_2x02_P2.54mm_Vertical_SMD, symbol Connector_Generic:Conn_02x02_Odd_Even
- added J103: ShittyAddOnR, Connector_PinSocket_2.54mm:PinSocket_2x02_P2.54mm_Vertical_SMD, symbol Connector_Generic:Conn_02x02_Odd_Even
- C101: renamed from C3; footprint (none) -> Capacitor_SMD:C_0805_2012Metric
- C102: renamed from C4; footprint (none) -> Capacitor_SMD:C_0805_2012Metric
- J104: renamed from J2; footprint Connector_PinHeader_1.00mm:PinHeader_2x20_P1.00mm_Vertical_SMD -> Connector_PinSocket_2.54mm:PinSocket_2x20_P2.54mm_Vertical_SMD
- J105: renamed from J8; footprint (none) -> Connector_PinHeader_1.00mm:PinHeader_1x02_P1.00mm_Horizontal
- SW107: renamed from SW7; value RESET -> ENTER
- TP101: renamed from TP1; footprint (none) -> TestPoint:TestPoint_Pad_D2.0mm
- TP102: renamed from TP2; footprint (none) -> TestPoint:TestPoint_Pad_D2.0mm
- TP103: renamed from TP3; footprint (none) -> TestPoint:TestPoint_Pad_D2.0mm
- TP104: renamed from TP4; footprint (none) -> TestPoint:TestPoint_Pad_D2.0mm
- TP105: renamed from TP5; footprint (none) -> TestPoint:TestPoint_Pad_D2.0mm
- TP106: renamed from TP6; footprint (none) -> TestPoint:TestPoint_Pad_D2.0mm
- TP107: renamed from TP7; footprint (none) -> TestPoint:TestPoint_Pad_D2.0mm
- TP108: renamed from TP8; footprint (none) -> TestPoint:TestPoint_Pad_D2.0mm
- Y101: renamed from Y1; footprint (none) -> Crystal:Crystal_SMD_MicroCrystal_CC4V-T1A-2Pin_5.0x1.9mm
- renumbered J3 to J101, R1 to R101, SW1 to SW101, SW2 to SW102, SW3 to SW103, SW4 to SW104, SW5 to SW105, SW6 to SW106, SW8 to SW108, U1 to U101
Connections:
- net labels added: AMP_SHUTDOWN, SCK_LED, SDA_LED
- wire segments 212 -> 231
- no-connect marks 47 -> 46
Other:
- note added: "DC27 BADGE - CPU, DISPLAY, USER INTERFACE - REV 1"
- note added: "Dual Shitty Add On’s!"
- note removed: "Am very unsure about this layout."
- note removed: "DC27 Audio Circuit\n"
- note removed: "ESD protection on power schematic"
- note removed: "Shitty Add On - 1\n"
- note removed: "Things to get from Bill:\nQSPI usage / pinout / where does it go\nWhere is I2C? Is it enabled?\nWhere do I2S Pins go?\nDo we need NFC pins?\nWhich SPI Bus is display on?\n\nIssue with cp2012n is it's sensitivity on vbus detect pin. If > 5.8v = boom"

Commit message: add pull ups to debug
Parts:
- added R102, R103: 10K, Resistor_SMD:R_0603_1608Metric, symbol Device:R
Connections:
- net labels added: DEBUG_SWO
- wire segments 231 -> 241
- no-connect marks 46 -> 44
Changed lines of the file:
@@
 P 1150 4500
 F 0 "J101" H 710 4546 50  0000 R CNN
-F 1 "Conn_ARM_JTAG_SWD_10" H 2150 3900 50  0000 R CNN
+F 1 "Conn_ARM_JTAG_SWD_10" V 850 4950 50  0000 R CNN
 F 2 "Connector_PinHeader_1.27mm:PinHeader_2x05_P1.27mm_Vertical_SMD" H 1200 3950 50  0001 L TNN
 F 3 "http://infocenter.arm.com/help/topic/com.arm.doc.faqs/attached/13634/cortex_debug_connectors.pdf" V 800 3250 50  0001 C CNN
@@
 Wire Wire Line
 	1150 3600 1150 3650
-Text GLabel 1850 4200 2    50   Output ~ 0
+Text GLabel 2300 4200 2    50   Output ~ 0
 ~RESET_TGTMCU
-Wire Wire Line
-	1650 4200 1850 4200
-Text GLabel 1850 4400 2    50   Output ~ 0
+Text GLabel 2300 4400 2    50   Output ~ 0
 DEBUG_SWDCLK
-Wire Wire Line
-	1650 4400 1850 4400
-Text GLabel 1850 4500 2    50   BiDi ~ 0
+Text GLabel 2300 4500 2    50   BiDi ~ 0
 DEBUG_SWDIO
-Wire Wire Line
-	1650 4500 1750 4500
 NoConn ~ 1650 4700
-NoConn ~ 1650 4600
 $Comp
 L Device:R R101
 U 1 1 5BB2FF77
 P 1750 3900
-F 0 "R101" H 1820 3946 50  0000 L CNN
-F 1 "10K" H 1820 3855 50  0000 L CNN
+F 0 "R101" H 1450 4000 50  0000 L CNN
+F 1 "10K" H 1500 3900 50  0000 L CNN
 F 2 "Resistor_SMD:R_0603_1608Metric" V 1680 3900 50  0001 C CNN
 F 3 "~" H 1750 3900 50  0001 C CNN
@@
 Wire Wire Line
 	1150 3650 1150 3900
-Wire Wire Line
-	1750 4050 1750 4500
-Connection ~ 1750 4500
-Wire Wire Line
-	1750 4500 1850 4500
 Text Notes 550  3350 0    50   ~ 10
 PROGRAMMING HEADER
@@
 Wire Wire Line
 	5750 4450 6000 4450
-NoConn ~ 5750 2750
 NoConn ~ 5750 4250
 NoConn ~ 5750 4150
@@
 	7200 1150 7200 1700
 Connection ~ 7200 1700
+Text GLabel 2300 4600 2    50   BiDi ~ 0
+DEBUG_SWO
+Wire Wire Line
+	1650 4200 2300 4200
+$Comp
+L Device:R R102
+U 1 1 5C3E5A2E
+P 1900 3900
+F 0 "R102" H 1970 3946 50  0000 L CNN
+F 1 "10K" H 1970 3855 50  0000 L CNN
+F 2 "Resistor_SMD:R_0603_1608Metric" V 1830 3900 50  0001 C CNN
+F 3 "~" H 1900 3900 50  0001 C CNN
+	1    1900 3900
+	1    0    0    -1
+$EndComp
+$Comp
+L Device:R R103
+U 1 1 5C3E5A7B
+P 2200 3900
+F 0 "R103" H 2270 3946 50  0000 L CNN
+F 1 "10K" H 2270 3855 50  0000 L CNN
+F 2 "Resistor_SMD:R_0603_1608Metric" V 2130 3900 50  0001 C CNN
+F 3 "~" H 2200 3900 50  0001 C CNN
+	1    2200 3900
+	1    0    0    -1
+$EndComp
+Wire Wire Line
+	1650 4600 2200 4600
+Wire Wire Line
+	1650 4400 1750 4400
+Wire Wire Line
+	1750 3650 1900 3650
+Wire Wire Line
+	1900 3650 1900 3750
+Connection ~ 1750 3650
+Wire Wire Line
+	1900 3650 2200 3650
+Wire Wire Line
+	2200 3650 2200 3750
+Connection ~ 1900 3650
+Wire Wire Line
+	2200 4050 2200 4600
+Connection ~ 2200 4600
+Wire Wire Line
+	2200 4600 2300 4600
+Wire Wire Line
+	1650 4500 1900 4500
+Wire Wire Line
+	1750 4050 1750 4400
+Connection ~ 1750 4400
+Wire Wire Line
+	1750 4400 2300 4400
+Wire Wire Line
+	1900 4050 1900 4500
+Connection ~ 1900 4500
+Wire Wire Line
+	1900 4500 2300 4500
+Text GLabel 6150 2750 2    50   BiDi ~ 0
+DEBUG_SWO
+Wire Wire Line
+	5750 2750 6150 2750
 $EndSCHEMATC
