File: hardware/dc27_badge_kicad/DC27_Switches.sch (KiCad schematic (older format))
At the start: 7 parts, among them SW801 SKRHAAE010, SW802 SKRHAAE010

Commit message: Check in V2 of the board. 0 unconnected nets, joypads on pcb
Parts:
- removed D801, D802, D803, D804, D805: BAT54AW, Package_TO_SOT_SMD:SOT-323_SC-70, symbol Diode:BAT54AW
- added D801, D802, D803, D804, D805, D806, D807, D808, D809, D810: BAT42W-V, Diode_SMD:D_SOD-123, symbol Diode:BAT42W-V
Connections:
- wire segments 66 -> 54
Other:
- note added: "1\n"
- note added: "4/12/2019\n"
- note added: "DC27 Badge - Joypad and Joypad Interrupt"
- note added: "Joypad Control\n"
- moved on the sheet: SW801, SW802
