File: hardware/dc27_badge_kicad/file5C2B533B.sch (KiCad schematic (older format))
At the start: 16 parts, among them J601 USB_MICRO_RIGHT, U601 CP2102N-A01-GQFN28

Commit message: add gerbers for prototype
Parts:
- removed L601, L602, L603: LXES15AAA1-153, Diode_SMD:D_01005_0402Metric, symbol jna_parts:LXES15AAA1-153
- added U602: TPD3E001DRLR, Package_TO_SOT_SMD:SOT-553, symbol DC27-badge-rescue:TPD3E001DRLR-Power_Protection
- U601: symbol Interface_USB:CP2102N-A01-GQFN24 -> DC27-badge-rescue:CP2102N-A01-GQFN24-Interface_USB
Connections:
- wire segments 77 -> 75
- no-connect marks 15 -> 16
Changed lines of the file:
@@
 	10250 2750 10000 2750
 $Comp
-L Interface_USB:CP2102N-A01-GQFN24 U601
+L DC27-badge-rescue:CP2102N-A01-GQFN24-Interface_USB U601
 U 1 1 5C2B55CC
 P 7350 3100
+AR Path="/5C2B55CC" Ref="U601"  Part="1"
+AR Path="/5C2B533C/5C2B55CC" Ref="U601"  Part="1"
 F 0 "U601" H 7350 3300 50  0000 C CNN
 F 1 "CP2102N-A01-GQFN28" H 7400 3150 50  0000 C CNN
@@
 Connection ~ 1500 1500
 Wire Wire Line
-	1500 1500 1850 1500
-Wire Wire Line
-	1300 1700 2250 1700
-Wire Wire Line
 	1400 2000 1400 2100
 Text Notes 700  2500 1    50   ~ 0
 floating shield to reduce noise
-$Comp
-L jna_parts:LXES15AAA1-153 L601
-U 1 1 5C4A6D96
-P 1850 2500
-F 0 "L601" V 1800 2600 50  0000 L CNN
-F 1 "LXES15AAA1-153" H 1600 2350 50  0000 L CNN
-F 2 "Diode_SMD:D_01005_0402Metric" H 1850 2500 50  0001 L BNN
-F 3 "LXES15AAA1-153" H 1850 2500 50  0001 L BNN
-F 4 "None" H 1850 2500 50  0001 L BNN "Field4"
-F 5 "0402 Murata" H 1850 2500 50  0001 L BNN "Field5"
-F 6 "Unavailable" H 1850 2500 50  0001 L BNN "Field6"
-F 7 "Murata" H 1850 2500 50  0001 L BNN "Field7"
-F 8 "ESD Suppressor TVS 4V 2-Pin Case 0402 T/R" H 1850 2500 50  0001 L BNN "Field8"
-	1    1850 2500
-	0    1    1    0
-$EndComp
-$Comp
-L jna_parts:LXES15AAA1-153 L602
-U 1 1 5C4A6E58
-P 2250 2500
-F 0 "L602" V 2200 2600 50  0000 L CNN
-F 1 "LXES15AAA1-153" H 2000 2350 50  0000 L CNN
-F 2 "Diode_SMD:D_01005_0402Metric" H 2250 2500 50  0001 L BNN
-F 3 "LXES15AAA1-153" H 2250 2500 50  0001 L BNN
-F 4 "None" H 2250 2500 50  0001 L BNN "Field4"
-F 5 "0402 Murata" H 2250 2500 50  0001 L BNN "Field5"
-F 6 "Unavailable" H 2250 2500 50  0001 L BNN "Field6"
-F 7 "Murata" H 2250 2500 50  0001 L BNN "Field7"
-F 8 "ESD Suppressor TVS 4V 2-Pin Case 0402 T/R" H 2250 2500 50  0001 L BNN "Field8"
-	1    2250 2500
-	0    1    1    0
-$EndComp
-$Comp
-L jna_parts:LXES15AAA1-153 L603
-U 1 1 5C4A6EA4
-P 2650 2500
-F 0 "L603" V 2600 2600 50  0000 L CNN
-F 1 "LXES15AAA1-153" H 2400 2350 50  0000 L CNN
-F 2 "Diode_SMD:D_01005_0402Metric" H 2650 2500 50  0001 L BNN
-F 3 "LXES15AAA1-153" H 2650 2500 50  0001 L BNN
-F 4 "None" H 2650 2500 50  0001 L BNN "Field4"
-F 5 "0402 Murata" H 2650 2500 50  0001 L BNN "Field5"
-F 6 "Unavailable" H 2650 2500 50  0001 L BNN "Field6"
-F 7 "Murata" H 2650 2500 50  0001 L BNN "Field7"
-F 8 "ESD Suppressor TVS 4V 2-Pin Case 0402 T/R" H 2650 2500 50  0001 L BNN "Field8"
-	1    2650 2500
-	0    1    1    0
-$EndComp
-Wire Wire Line
-	2650 2300 2650 1800
-Wire Wire Line
-	1300 1800 2650 1800
-Connection ~ 2650 1800
-Wire Wire Line
-	2650 1800 2800 1800
-Wire Wire Line
-	2250 2300 2250 1700
-Connection ~ 2250 1700
-Wire Wire Line
-	2250 1700 2800 1700
-Wire Wire Line
-	1850 2300 1850 1500
-Connection ~ 1850 1500
-$Comp
-L power:GND #PWR0606
-U 1 1 5C4AA6BD
-P 2250 3100
-F 0 "#PWR0606" H 2250 2850 50  0001 C CNN
-F 1 "GND" H 2255 2927 50  0000 C CNN
-F 2 "" H 2250 3100 50  0001 C CNN
-F 3 "" H 2250 3100 50  0001 C CNN
-	1    2250 3100
-	1    0    0    -1
-$EndComp
-Wire Wire Line
-	1850 2700 1850 3050
-Wire Wire Line
-	1850 3050 2250 3050
-Wire Wire Line
-	2650 3050 2650 2700
-Wire Wire Line
-	2250 3100 2250 3050
-Connection ~ 2250 3050
-Wire Wire Line
-	2250 3050 2650 3050
-Wire Wire Line
-	2250 3050 2250 2700
 Text GLabel 4750 2750 1    50   Input ~ 0
 VBUS
 Wire Wire Line
 	4750 2750 4750 3150
-Wire Wire Line
-	1850 1500 3650 1500
 $Comp
 L Device:C C601
@@
 Wire Wire Line
 	4150 1500 4350 1500
-Text Notes 2700 2850 0    50   ~ 0
+Text Notes 3150 2850 0    50   ~ 0
 ESD Protection\n
 NoConn ~ 6550 2850
@@
 Wire Wire Line
 	6400 3050 6400 3300
+$Comp
+L DC27-badge-rescue:TPD3E001DRLR-Power_Protection U602
+U 1 1 5C6C8281
+P 2450 2850
+F 0 "U602" V 2750 2400 50  0000 L CNN
+F 1 "TPD3E001DRLR" V 2650 2050 50  0000 L CNN
+F 2 "Package_TO_SOT_SMD:SOT-553" H 1750 2550 50  0001 C CNN
+F 3 "" H 2250 3100 50  0001 C CNN
+	1    2450 2850
+	0    -1   -1   0
+$EndComp
+Wire Wire Line
+	1500 1500 1750 1500
+$Comp
+L power:GND #PWR0114
+U 1 1 5C6C877C
+P 2900 2950
+F 0 "#PWR0114" H 2900 2700 50  0001 C CNN
+F 1 "GND" H 2905 2777 50  0000 C CNN
+F 2 "" H 2900 2950 50  0001 C CNN
+F 3 "" H 2900 2950 50  0001 C CNN
+	1    2900 2950
+	1    0    0    -1
+$EndComp
+Wire Wire Line
+	2900 2850 2900 2950
+Wire Wire Line
+	2750 2850 2900 2850
+Wire Wire Line
+	2450 3250 2450 3450
+Wire Wire Line
+	2450 3450 1750 3450
+Wire Wire Line
+	1750 3450 1750 1500
+Connection ~ 1750 1500
+Wire Wire Line
+	1750 1500 3650 1500
+Wire Wire Line
+	1300 1800 2450 1800
+NoConn ~ 2550 2450
+Wire Wire Line
+	2350 2450 2350 1700
+Wire Wire Line
+	1300 1700 2350 1700
+Connection ~ 2350 1700
+Wire Wire Line
+	2350 1700 2800 1700
+Wire Wire Line
+	2450 1800 2450 2450
+Connection ~ 2450 1800
+Wire Wire Line
+	2450 1800 2800 1800
 $EndSCHEMATC

Commit message: add AST-01078 3d model and kicad footprint, check in current budget, update charging circut to MCP73833 instead of MCP73831:
Parts:
- J601: symbol MF_Connectors:USB_MICRO_RIGHT -> DC27-badge-rescue:USB_MICRO_RIGHT-MF_Connectors-DC27-badge-rescue
Changed lines of the file:
@@
 EESchema Schematic File Version 4
 LIBS:DC27-badge-cache
-EELAYER 26 0
+EELAYER 29 0
 EELAYER END
 $Descr A4 11693 8268
@@
 Wire Wire Line
 	1400 2000 1300 2000
-$Comp
-L power:PWR_FLAG #FLG?
-U 1 1 5C4486B1
-P 1500 1300
-AR Path="/5BA3F217/5C4486B1" Ref="#FLG?"  Part="1"
-AR Path="/5C2B533C/5C4486B1" Ref="#FLG0601"  Part="1"
-F 0 "#FLG0601" H 1500 1375 50  0001 C CNN
-F 1 "PWR_FLAG" H 1500 1474 50  0000 C CNN
-F 2 "" H 1500 1300 50  0001 C CNN
-F 3 "~" H 1500 1300 50  0001 C CNN
-	1    1500 1300
-	1    0    0    -1
-$EndComp
 Text GLabel 4350 1500 2    50   Output ~ 0
 VBUS
 $Comp
-L MF_Connectors:USB_MICRO_RIGHT J?
+L DC27-badge-rescue:USB_MICRO_RIGHT-MF_Connectors-DC27-badge-rescue J?
 U 1 1 5C44869C
 P 1000 1800
 AR Path="/5BA3F217/5C44869C" Ref="J?"  Part="1"
 AR Path="/5C2B533C/5C44869C" Ref="J601"  Part="1"
+AR Path="/5C44869C" Ref="J601"  Part="1"
 F 0 "J601" H 1056 2254 45  0000 C CNN
 F 1 "USB_MICRO_RIGHT" H 1056 2170 45  0000 C CNN
@@
 Wire Wire Line
 	1300 1600 1450 1600
-Wire Wire Line
-	1450 1500 1500 1500
-Wire Wire Line
-	1500 1300 1500 1500
-Connection ~ 1500 1500
 Wire Wire Line
 	1400 2000 1400 2100
@@
 $EndComp
 Wire Wire Line
-	1500 1500 1750 1500
-$Comp
-L power:GND #PWR0114
-U 1 1 5C6C877C
-P 2900 2950
-F 0 "#PWR0114" H 2900 2700 50  0001 C CNN
-F 1 "GND" H 2905 2777 50  0000 C CNN
-F 2 "" H 2900 2950 50  0001 C CNN
-F 3 "" H 2900 2950 50  0001 C CNN
-	1    2900 2950
-	1    0    0    -1
-$EndComp
-Wire Wire Line
-	2900 2850 2900 2950
-Wire Wire Line
-	2750 2850 2900 2850
-Wire Wire Line
 	2450 3250 2450 3450
 Wire Wire Line
@@
 Connection ~ 1750 1500
 Wire Wire Line
-	1750 1500 3650 1500
-Wire Wire Line
 	1300 1800 2450 1800
 NoConn ~ 2550 2450
@@
 Wire Wire Line
 	2450 1800 2800 1800
+Wire Wire Line
+	1450 1500 1550 1500
+Wire Wire Line
+	1750 1500 3650 1500
+$Comp
+L power:PWR_FLAG #FLG0101
+U 1 1 5CC5F3C8
+P 1550 1400
+F 0 "#FLG0101" H 1550 1475 50  0001 C CNN
+F 1 "PWR_FLAG" H 1550 1573 50  0000 C CNN
+F 2 "" H 1550 1400 50  0001 C CNN
+F 3 "~" H 1550 1400 50  0001 C CNN
+	1    1550 1400
+	1    0    0    -1
+$EndComp
+Wire Wire Line
+	1550 1400 1550 1500
+Connection ~ 1550 1500
+Wire Wire Line
+	1550 1500 1750 1500
+$Comp
+L power:GND #PWR0114
+U 1 1 5CCAE9BD
+P 3000 3000
+F 0 "#PWR0114" H 3000 2750 50  0001 C CNN
+F 1 "GND" H 3005 2827 50  0000 C CNN
+F 2 "" H 3000 3000 50  0001 C CNN
+F 3 "" H 3000 3000 50  0001 C CNN
+	1    3000 3000
+	1    0    0    -1
+$EndComp
+Wire Wire Line
+	3000 2850 3000 3000
+Wire Wire Line
+	2750 2850 3000 2850
 $EndSCHEMATC

Commit message: Fix R604 and other dumb 0603/0805 mistakes
Parts:
- R604: footprint Resistor_SMD:R_0603_1608Metric -> Resistor_SMD:R_0805_2012Metric
Changed lines of the file:
@@
 F 0 "R604" H 4820 3346 50  0000 L CNN
 F 1 "22.1k" H 4820 3255 50  0000 L CNN
-F 2 "Resistor_SMD:R_0603_1608Metric" V 4680 3300 50  0001 C CNN
+F 2 "Resistor_SMD:R_0805_2012Metric" V 4680 3300 50  0001 C CNN
 F 3 "~" H 4750 3300 50  0001 C CNN
 	1    4750 3300
